Commit message: multi

File: unitree_go2_description/urdf/lidar_4D_lidar.xacro (robot description, xacro)
@@ -35,5 +35,5 @@
     <gazebo reference="lidar_l1_link">
         <sensor name="lidar_l1" type="gpu_lidar">
-            <topic>unitree_lidar</topic>
+            <topic>${ns_prefix}/unitree_lidar</topic>
             <update_rate>10</update_rate>
             <lidar>

File: unitree_go2_description/urdf/unitree_go2_gazebo.xacro (robot description, xacro)
@@ -25,6 +25,11 @@
   <gazebo>
     <plugin filename="gz_ros2_control-system" name="gz_ros2_control::GazeboSimROS2ControlPlugin">
-      <parameters>$(find unitree_go2_sim)/config/ros_control/ros_control.yaml</parameters>
+	      <!-- Do not rely on $(find ...) resolution in Gazebo. Launch should pass an absolute path. -->
+	      <parameters>$(arg ros2_control_params)</parameters>
       <robot_param_node>robot_state_publisher</robot_param_node>
+      <!-- Namespace the controller manager and ROS interfaces per robot. -->
+      <ros>
+        <namespace>$(arg robot_namespace)</namespace>
+      </ros>
     </plugin>
   </gazebo>
@@ -34,5 +39,5 @@
       <odom_frame>odom</odom_frame>
       <robot_base_frame>base_link</robot_base_frame>
-      <odom_topic>/odom</odom_topic>
+      <odom_topic>${ns_prefix}/odom</odom_topic>
       <odom_publish_frequency>50</odom_publish_frequency>
     </plugin>
@@ -44,5 +49,5 @@
       <update_rate>100</update_rate>
       <visualize>true</visualize>
-      <topic>imu/data</topic>
+      <topic>${ns_prefix}/imu/data</topic>
       <gz_frame_id>imu_link</gz_frame_id>
       <imu>
@@ -112,5 +117,5 @@
       <update_rate>10</update_rate>
       <visualize>1</visualize>
-      <topic>rgb_image</topic>
+      <topic>${ns_prefix}/rgb_image</topic>
     </sensor>
   </gazebo>

File: unitree_go2_description/urdf/unitree_go2_robot.xacro (robot description, xacro)
@@ -1,6 +1,20 @@
 <?xml version="1.0"?>
-<robot name="go2"
+<robot name="$(arg robot_name)"
     xmlns:xacro="http://www.ros.org/wiki/xacro">
     <xacro:arg name="DEBUG" default="false"/>
+    <!-- Used for multi-robot launches. -->
+    <xacro:arg name="robot_name" default="go2"/>
+    <xacro:arg name="robot_namespace" default=""/>
+    <!-- Path to ros2_control controller configuration. Launch should override with an absolute path. -->
+    <xacro:arg name="ros2_control_params" default="$(find unitree_go2_sim)/config/ros_control/ros_control.yaml"/>
+    <!--
+      Xacro <arg> does not automatically create a python variable.
+      We must explicitly copy the arg value into a property before using it
+      inside ${...} expressions.
+    -->
+    <xacro:property name="robot_namespace" value="$(arg robot_namespace)"/>
+    <xacro:property name="robot_name" value="$(arg robot_name)"/>
+    <!-- Convenience prefix for Gazebo Sim and ROS topic names. -->
+    <xacro:property name="ns_prefix" value="${'/' + robot_namespace if robot_namespace else ''}"/>
     <xacro:include filename="$(find unitree_go2_description)/urdf/const.xacro"/>
     <xacro:include filename="$(find unitree_go2_description)/urdf/materials.xacro"/>

File: unitree_go2_description/urdf/velodyne.xacro (robot description, xacro)
@@ -50,5 +50,5 @@
     <gazebo reference="velodyne">
         <sensor name="velodyne-VLP16" type="gpu_lidar">
-            <topic>velodyne_points</topic>
+            <topic>${ns_prefix}/velodyne_points</topic>
             <update_rate>10</update_rate>
             <gz_frame_id>velodyne</gz_frame_id>
